Commit message: creation of the urdf description files for the dextrobot

File: ROS/dextrobot_ws/src/dextrobot_description/src/robot/dextrobot.urdf.xacro (robot description, xacro)
@@ -6,8 +6,7 @@
 	<!-- First we import all posible elements defined in the urdf.xacro files. All these elements are defined as macro:xacros -->
 	<!-- Import summit XL base elements -->
-	<xacro:include filename="$(find summit_xl_description)/urdf/bases/summit_xl_base.urdf.xacro" />
+	<xacro:include filename="$(find dextrobot_description)/src/urdf/bases/dextrobot_base.urdf.xacro" />
 	<!-- Import summit XL wheels -->
-	<xacro:include filename="$(find summit_xl_description)/urdf/wheels/rubber_wheel.urdf.xacro" />
-    <xacro:include filename="$(find summit_xl_description)/urdf/wheels/omni_wheel.urdf.xacro" />
+    <xacro:include filename="$(find dextrobot_description)/src/urdf/wheels/omni_wheel.urdf.xacro" />
 	<!-- Import all available sensors -->
 	<xacro:include filename="$(find robotnik_sensors)/urdf/all_sensors.urdf.xacro" />
@@ -19,9 +18,9 @@
 	<!-- Flag to select the high or low quality model -->
 	<xacro:property name="hq" value="true" />
-	<xacro:arg name="prefix" default="summit_xl_"/>
+	<xacro:arg name="prefix" default="dextrobot_"/>
 	<xacro:arg name="ros_planar_move_plugin" default="false"/>
 	<xacro:arg name="omni_wheels" default="false"/>
 	<xacro:arg name="gpu" default="false"/>
-    <xacro:macro name="summit_xl" params="prefix publish_bf hq">
+    <xacro:macro name="dextrobot" params="prefix publish_bf hq">
 		<!-- *************** -->
 		<!-- Robots Elements -->
@@ -30,18 +29,4 @@
 		<!-- Summit XL base -->
 		<xacro:summit_xl_base prefix="$(arg prefix)" publish_bf="true" hq="${hq}" />
-    <xacro:unless value="$(arg omni_wheels)">
-  		<xacro:rubber_wheel prefix="$(arg prefix)front_right" parent="$(arg prefix)base_link" reflect="false" hq="${hq}">
-  			<origin xyz="${wheel_offset_x} -${wheel_offset_y} ${wheel_offset_z}" rpy="0 0 0"/>
-  		</xacro:rubber_wheel>
-  		<xacro:rubber_wheel prefix="$(arg prefix)front_left" parent="$(arg prefix)base_link" reflect="true" hq="${hq}">
-  			<origin xyz="${wheel_offset_x} ${wheel_offset_y} ${wheel_offset_z}" rpy="0 0 0"/>
-  		</xacro:rubber_wheel>
-  		<xacro:rubber_wheel prefix="$(arg prefix)back_left" parent="$(arg prefix)base_link" reflect="true" hq="${hq}">
-  			<origin xyz="-${wheel_offset_x} ${wheel_offset_y} ${wheel_offset_z}" rpy="0 0 0"/>
-  		</xacro:rubber_wheel>
-  		<xacro:rubber_wheel prefix="$(arg prefix)back_right" parent="$(arg prefix)base_link" reflect="false" hq="${hq}">
-  			<origin xyz="-${wheel_offset_x} -${wheel_offset_y} ${wheel_offset_z}" rpy="0 0 0"/>
-  		</xacro:rubber_wheel>
-    </xacro:unless>
     <xacro:if value="$(arg omni_wheels)">
   		<xacro:omni_wheel prefix="$(arg prefix)front_right" parent="$(arg prefix)base_link" reflect="false" hq="${hq}">
@@ -66,16 +51,8 @@
 			<origin xyz="0.0 0.0 0.33" rpy="0 0 0"/>
 		</xacro:sensor_hokuyo_ust10lx>
-		<!-- ptz camera -->
-		<xacro:sensor_axis prefix="$(arg prefix)front_ptz_camera" parent="$(arg prefix)base_link">
-			<origin xyz="0.19 0 0.26" rpy="0 ${15*PI/180} 0"/>
-		</xacro:sensor_axis>
-	  <!-- RGBD -->
-	  <xacro:sensor_orbbec_astra prefix="$(arg prefix)front_rgbd_camera" parent="$(arg prefix)base_link" prefix_topic="front_rgbd_camera">
+	    <!-- RGBD -->
+	    <xacro:sensor_orbbec_astra prefix="$(arg prefix)front_rgbd_camera" parent="$(arg prefix)base_link" prefix_topic="front_rgbd_camera">
 			<origin xyz="0.324 0.012 0.172" rpy="0 0 0"/>
 		</xacro:sensor_orbbec_astra>
-	  <!-- GPS -->
-	  <xacro:sensor_gps prefix="$(arg prefix)gps" parent="$(arg prefix)base_link">
-			<origin xyz="-0.22 0 0.275" rpy="0 0 0"/>
-		</xacro:sensor_gps>
    </xacro:macro>
    <!-- Gazebo ros control pluggins -->
@@ -85,7 +62,4 @@
 			<xacro:omni_steering prefix="$(arg prefix)" publish_tf="true"/>
 		</xacro:if>
-		<xacro:unless value="$(arg omni_wheels)">
-			<xacro:skid_steering prefix="$(arg prefix)" publish_tf="true"/>
-		</xacro:unless>
 	</xacro:if>
    <xacro:summit_xl prefix="$(arg prefix)" publish_bf="true" hq="true"/>

File: ROS/dextrobot_ws/src/dextrobot_description/src/urdf/wheels/omni_wheel.urdf.xacro (robot description, xacro)
@@ -3,7 +3,7 @@
   <xacro:property name="M_PI" value="3.1415926535897931" />
   <!-- Wheels -->
-  <xacro:property name="omni_wheel_radius" value="0.127" />
-  <xacro:property name="omni_wheel_height" value="0.087" />
-  <xacro:property name="omni_wheel_mass" value="6.5" /> <!-- in kg-->
+  <xacro:property name="omni_wheel_radius" value="0.04" />
+  <xacro:property name="omni_wheel_height" value="0.04" />
+  <xacro:property name="omni_wheel_mass" value="0.7" /> <!-- in kg-->
   <xacro:macro name="cylinder_inertia" params="m r h">
     <inertia  ixx="${m*(3*r*r+h*h)/12}" ixy = "0" ixz = "0"
@@ -26,10 +26,10 @@
           <xacro:if value="${reflect}">
             <geometry>
-              <mesh filename="package://summit_xl_description/meshes/wheels/omni_wheel_1.dae" />
+              <mesh filename="package://dextrobot_description/src/meshes/wheels/mechanum_wheel_1.dae" />
             </geometry>
           </xacro:if>
           <xacro:unless value="${reflect}">
             <geometry>
-              <mesh filename="package://summit_xl_description/meshes/wheels/omni_wheel_2.dae" />
+              <mesh filename="package://summit_xl_description/meshes/wheels/mechanum_wheel_2.dae" />
             </geometry>
 		  </xacro:unless>
@@ -48,14 +48,5 @@
 				<origin xyz="0 0 0" rpy="${PI/2} 0 0" />
         <geometry>
-          <!--sphere radius="${omni_wheel_radius}" /-->
-<!--
-          <xacro:if value="${reflect}">
-              <mesh filename="package://summit_xl_description/meshes/wheels/omni_wheel_1.dae" />
-          </xacro:if>
-          <xacro:unless value="${reflect}">
-              <mesh filename="package://summit_xl_description/meshes/wheels/omni_wheel_2.dae" />
-					</xacro:unless>
--->
-					<cylinder length="${omni_wheel_height}" radius="${omni_wheel_radius}" />
+				<cylinder length="${omni_wheel_height}" radius="${omni_wheel_radius}" />
         </geometry>
       </collision>

Commit message: small changes to make the launch file work

File: ROS/dextrobot_ws/src/dextrobot_description/src/robot/dextrobot.urdf.xacro (robot description, xacro)
@@ -28,5 +28,5 @@
 		<!-- Here we create the robot elements using the xacro:macros imported at the beggining of this file -->
 		<!-- Summit XL base -->
-		<xacro:summit_xl_base prefix="$(arg prefix)" publish_bf="true" hq="${hq}" />
+		<xacro:dextrobot_base prefix="$(arg prefix)" publish_bf="true" hq="${hq}" />
     <xacro:if value="$(arg omni_wheels)">
   		<xacro:omni_wheel prefix="$(arg prefix)front_right" parent="$(arg prefix)base_link" reflect="false" hq="${hq}">
@@ -48,5 +48,5 @@
 		</xacro:sensor_imu>
 		<!-- 2d laser -->
-		<xacro:sensor_hokuyo_ust10lx prefix="$(arg prefix)front_laser" parent="$(arg prefix)base_link" prefix_topic="front_laser" gpu="$(arg gpu)">
+		<xacro:sensor_hokuyo_ust10lx prefix="$(arg prefix)front_laser" parent="$(arg prefix)base_link" prefix_topic="front_laser">
 			<origin xyz="0.0 0.0 0.33" rpy="0 0 0"/>
 		</xacro:sensor_hokuyo_ust10lx>
@@ -63,4 +63,4 @@
 		</xacro:if>
 	</xacro:if>
-   <xacro:summit_xl prefix="$(arg prefix)" publish_bf="true" hq="true"/>
+   <xacro:dextrobot prefix="$(arg prefix)" publish_bf="true" hq="true"/>
 </robot>

File: ROS/dextrobot_ws/src/dextrobot_description/src/urdf/bases/dextrobot_base.urdf.xacro (robot description, xacro)
@@ -27,4 +27,5 @@
       <mass value="125.0" />
       <origin xyz="0 0 0" />
+    </inertial>
     <visual>
       <origin xyz="0 0 0" rpy="0 0 0" />

Commit message: added robot description and visualization in RVIZ

File: ROS/dextrobot_ws/src/dextrobot_description/src/robot/dextrobot.urdf.xacro (robot description, xacro)
@@ -1,4 +1,4 @@
 <?xml version="1.0"?>
-<robot name="summit_xl" xmlns:xacro="http://wiki.ros.org/xacro">
+<robot name="dextrobot" xmlns:xacro="http://wiki.ros.org/xacro">
 	<!-- ***************** -->
 	<!-- Imported elements -->
@@ -13,13 +13,49 @@
 	<xacro:property name="PI" value="3.1415926535897931"/>
 	<!-- Wheel parameters -->
-	<xacro:property name="wheel_offset_x" value="0.229" />    <!-- x,y,z in translation from base_link to the center of the wheel -->
-	<xacro:property name="wheel_offset_y" value="0.235" />
-	<xacro:property name="wheel_offset_z" value="0.0" />
+	<!-- Front Left -->
+	<xacro:property name="wheel_1_offset_x" value="-1" />    <!-- x,y,z in translation from base_link to the center of the wheel -->
+	<xacro:property name="wheel_1_offset_y" value="-0.8" />
+	<xacro:property name="wheel_1_offset_z" value="0.0" />
+	<!-- Front Right -->
+	<xacro:property name="wheel_2_offset_x" value="0.72" />    <!-- x,y,z in translation from base_link to the center of the wheel -->
+	<xacro:property name="wheel_2_offset_y" value="0.05" />
+	<xacro:property name="wheel_2_offset_z" value="0.0" />
+	<!-- Back Left -->
+	<xacro:property name="wheel_3_offset_x" value="-1" />    <!-- x,y,z in translation from base_link to the center of the wheel -->
+	<xacro:property name="wheel_3_offset_y" value="-2.2" />
+	<xacro:property name="wheel_3_offset_z" value="0.0" />
+	<!-- Back Right -->
+	<xacro:property name="wheel_4_offset_x" value="0.72" />    <!-- x,y,z in translation from base_link to the center of the wheel -->
+	<xacro:property name="wheel_4_offset_y" value="-1.35" />
+	<xacro:property name="wheel_4_offset_z" value="0.0" />
+	<!-- IMU parameters -->
+	<xacro:property name="imu_offset_x" value="0.229" />    <!-- x,y,z in translation from base_link to the center of the wheel -->
+	<xacro:property name="imu_offset_y" value="0.235" />
+	<xacro:property name="imu_offset_z" value="0.0" />
+	<!-- Camera parameters -->
+	<xacro:property name="camera_offset_x" value="-0.15" />    <!-- x,y,z in translation from base_link to the center of the wheel -->
+	<xacro:property name="camera_offset_y" value="-0.25" />
+	<xacro:property name="camera_offset_z" value="1.1" />
+	<!-- Sonar parameters -->
+	<!-- front sonar -->
+	<xacro:property name="front_sonar_offset_x" value="0.229" />    <!-- x,y,z in translation from base_link to the center of the wheel -->
+	<xacro:property name="front_sonar_offset_y" value="0.235" />
+	<xacro:property name="front_sonar_offset_z" value="0.0" />
+	<!-- left sonar -->
+	<xacro:property name="left_sonar_offset_x" value="0.229" />    <!-- x,y,z in translation from base_link to the center of the wheel -->
+	<xacro:property name="left_sonar_offset_y" value="0.235" />
+	<xacro:property name="left_sonar_offset_z" value="0.0" />
+	<!-- right sonar -->
+	<xacro:property name="right_sonar_offset_x" value="0.229" />    <!-- x,y,z in translation from base_link to the center of the wheel -->
+	<xacro:property name="right_sonar_offset_y" value="0.235" />
+	<xacro:property name="right_sonar_offset_z" value="0.0" />
+	<!-- back sonar -->
+	<xacro:property name="back_sonar_offset_x" value="0.229" />    <!-- x,y,z in translation from base_link to the center of the wheel -->
+	<xacro:property name="back_sonar_offset_y" value="0.235" />
+	<xacro:property name="back_sonar_offset_z" value="0.0" />
 	<!-- Flag to select the high or low quality model -->
 	<xacro:property name="hq" value="true" />
 	<xacro:arg name="prefix" default="dextrobot_"/>
-	<xacro:arg name="ros_planar_move_plugin" default="false"/>
-	<xacro:arg name="omni_wheels" default="false"/>
-	<xacro:arg name="gpu" default="false"/>
+	<xacro:arg name="ros_planar_move_plugin" default="true"/>
     <xacro:macro name="dextrobot" params="prefix publish_bf hq">
 		<!-- *************** -->
@@ -29,29 +65,23 @@
 		<!-- Summit XL base -->
 		<xacro:dextrobot_base prefix="$(arg prefix)" publish_bf="true" hq="${hq}" />
-    <xacro:if value="$(arg omni_wheels)">
+		<xacro:omni_wheel prefix="$(arg prefix)front_left" parent="$(arg prefix)base_link" reflect="false" hq="${hq}">
+  			<origin xyz="${wheel_1_offset_x} ${wheel_1_offset_y} ${wheel_1_offset_z}" rpy="0 0 0"/>
+  		</xacro:omni_wheel>
   		<xacro:omni_wheel prefix="$(arg prefix)front_right" parent="$(arg prefix)base_link" reflect="false" hq="${hq}">
-  			<origin xyz="${wheel_offset_x} -${wheel_offset_y} ${wheel_offset_z}" rpy="0 0 0"/>
-  		</xacro:omni_wheel>
-  		<xacro:omni_wheel prefix="$(arg prefix)front_left" parent="$(arg prefix)base_link" reflect="true" hq="${hq}">
-  			<origin xyz="${wheel_offset_x} ${wheel_offset_y} ${wheel_offset_z}" rpy="0 0 0"/>
+  			<origin xyz="${wheel_2_offset_x} ${wheel_2_offset_y} ${wheel_2_offset_z}" rpy="0 0 ${PI}"/>
   		</xacro:omni_wheel>
   		<xacro:omni_wheel prefix="$(arg prefix)back_left" parent="$(arg prefix)base_link" reflect="true" hq="${hq}">
-  			<origin xyz="-${wheel_offset_x} ${wheel_offset_y} ${wheel_offset_z}" rpy="0 0 0"/>
+  			<origin xyz="${wheel_3_offset_x} ${wheel_3_offset_y} ${wheel_3_offset_z}" rpy="0 0 0"/>
   		</xacro:omni_wheel>
   		<xacro:omni_wheel prefix="$(arg prefix)back_right" parent="$(arg prefix)base_link" reflect="false" hq="${hq}">
-  			<origin xyz="-${wheel_offset_x} -${wheel_offset_y} ${wheel_offset_z}" rpy="0 0 0"/>
+  			<origin xyz="${wheel_4_offset_x} ${wheel_4_offset_y} ${wheel_4_offset_z}" rpy="0 0 ${PI}"/>
   		</xacro:omni_wheel>
-    </xacro:if>
         <!-- IMU -->
-		<xacro:sensor_imu prefix="$(arg prefix)imu" parent="$(arg prefix)base_link">
-			<origin xyz="-0.18 0.0 0.170" rpy="0 0 0"/>
-		</xacro:sensor_imu>
-		<!-- 2d laser -->
-		<xacro:sensor_hokuyo_ust10lx prefix="$(arg prefix)front_laser" parent="$(arg prefix)base_link" prefix_topic="front_laser">
-			<origin xyz="0.0 0.0 0.33" rpy="0 0 0"/>
-		</xacro:sensor_hokuyo_ust10lx>
+		<xacro:sensor_imu_hector prefix="$(arg prefix)imu" parent="$(arg prefix)base_link">
+			<origin xyz="${imu_offset_x} ${imu_offset_y} ${imu_offset_z}" rpy="0 0 0"/>
+		</xacro:sensor_imu_hector>
 	    <!-- RGBD -->
 	    <xacro:sensor_orbbec_astra prefix="$(arg prefix)front_rgbd_camera" parent="$(arg prefix)base_link" prefix_topic="front_rgbd_camera">
-			<origin xyz="0.324 0.012 0.172" rpy="0 0 0"/>
+			<origin xyz="${camera_offset_x} ${camera_offset_y} ${camera_offset_z}" rpy="0 0 ${PI/2}"/>
 		</xacro:sensor_orbbec_astra>
    </xacro:macro>
@@ -59,7 +89,5 @@
    <xacro:ros_control/>
 	<xacro:if value="$(arg ros_planar_move_plugin)">
-		<xacro:if value="$(arg omni_wheels)">
-			<xacro:omni_steering prefix="$(arg prefix)" publish_tf="true"/>
-		</xacro:if>
+		<xacro:omni_steering prefix="$(arg prefix)" publish_tf="true"/>
 	</xacro:if>
    <xacro:dextrobot prefix="$(arg prefix)" publish_bf="true" hq="true"/>

File: ROS/dextrobot_ws/src/dextrobot_description/src/urdf/bases/dextrobot_base.gazebo.xacro (robot description, xacro)
@@ -13,25 +13,4 @@
     </gazebo>
 	</xacro:macro>
-	<!-- skid steering plugin -->
-	<xacro:macro name="skid_steering" params="prefix publish_tf">
-    <gazebo>
-      <plugin name="skid_steer_drive_controller" filename="libgazebo_ros_skid_steer_drive.so">
-			<!--<robotNamespace>/summit_xl</robotNamespace>-->
-		    <updateRate>50.0</updateRate>
-		    <leftFrontJoint>${prefix}front_left_wheel_joint</leftFrontJoint>
-		    <rightFrontJoint>${prefix}front_right_wheel_joint</rightFrontJoint>
-		    <leftRearJoint>${prefix}back_left_wheel_joint</leftRearJoint>
-		    <rightRearJoint>${prefix}back_right_wheel_joint</rightRearJoint>
-		    <wheelSeparation>0.462</wheelSeparation>
-		    <wheelDiameter>0.08</wheelDiameter>
-		    <robotBaseFrame>${prefix}base_footprint</robotBaseFrame>
-		    <torque>50</torque>
-		    <commandTopic>dextrobot_base_control/cmd_vel</commandTopic>
-		    <odometryTopic>dextrobot_base_control/odom</odometryTopic>
-		    <odometryFrame>${prefix}odom</odometryFrame>
-		    <broadcastTF>${publish_tf}</broadcastTF>
-      </plugin>
-    </gazebo>
-  </xacro:macro>
   <xacro:macro name="omni_steering" params="prefix publish_tf">
 		<gazebo>
@@ -46,17 +25,4 @@
 	  </gazebo>
   </xacro:macro>
-  	<xacro:macro name="skid_steering" params="prefix publish_tf">
-		<gazebo>
-			<plugin name="skid_steering" filename="libgazebo_ros_planar_move.so">
-			<commandTopic>dextrobot_base_control/cmd_vel</commandTopic>
-			<odometryTopic>dextrobot_base_control/odom</odometryTopic>
-			<odometryFrame>${prefix}odom</odometryFrame>
-			<odometryRate>50.0</odometryRate>
-			<robotBaseFrame>${prefix}base_footprint</robotBaseFrame>
-			<publishTF>${publish_tf}</publishTF>
-			<enableYAxis>false</enableYAxis>
-			</plugin>
-		</gazebo>
-  	</xacro:macro>
   <xacro:macro name="ros_force_based_move" params="publish_tf prefix">
 	  <gazebo>

File: ROS/dextrobot_ws/src/dextrobot_description/src/urdf/bases/dextrobot_base.urdf.xacro (robot description, xacro)
@@ -1,4 +1,4 @@
 <?xml version="1.0"?>
-<robot name="summit_xl" xmlns:xacro="http://wiki.ros.org/xacro">
+<robot name="dextrobot" xmlns:xacro="http://wiki.ros.org/xacro">
   <xacro:include filename="$(find dextrobot_description)/src/urdf/bases/dextrobot_base.gazebo.xacro" />
   <xacro:macro name="dextrobot_base" params="prefix publish_bf hq">
@@ -24,18 +24,14 @@
   <!-- BASE_LINK -->
   <link name="${prefix}base_link">
-    <inertial>
-      <mass value="125.0" />
-      <origin xyz="0 0 0" />
-    </inertial>
     <visual>
-      <origin xyz="0 0 0" rpy="0 0 0" />
+      <origin xyz="2 0 0.1" rpy="${PI/2} 0 ${-PI/2}" />
       <xacro:if value="${hq}">
       <geometry>
-      <mesh filename="package://dextrobot_description/src/mesh/base/dextrobot_chassis.stl"/>
+      <mesh filename="package://dextrobot_description/src/mesh/base/dextrobot_chassis.STL" scale="0.01 0.01 0.01"/>
       </geometry>
       </xacro:if>
       <xacro:unless value="${hq}">
       <geometry>
-      <mesh filename="package://dextrobot_description/src/mesh/base/dextrobot_chassis.dae"/>
+      <mesh filename="package://dextrobot_description/src/mesh/base/dextrobot_chassis.dae" scale="0.01 0.01 0.01"/>
       </geometry>
       </xacro:unless>
@@ -45,13 +41,10 @@
     </visual>
     <collision>
-       <origin xyz="0 0 0" rpy="0 0 0 " />
+       <origin xyz="2 0 0.1" rpy="${PI/2} 0 ${-PI/2}" />
        <geometry>
-         <mesh filename="package://dextrobot_description/src/mesh/base/dextrobot_chassis.dae"/>
+         <mesh filename="package://dextrobot_description/src/mesh/base/dextrobot_chassis.dae" scale="0.01 0.01 0.01"/>
        </geometry>
     </collision>
   </link>
-  <gazebo reference="${prefix}base_link">
-    <material>Gazebo/Black</material>
-  </gazebo>
   </xacro:macro>
 </robot>

File: ROS/dextrobot_ws/src/dextrobot_description/src/urdf/wheels/omni_wheel.urdf.xacro (robot description, xacro)
@@ -5,5 +5,5 @@
   <xacro:property name="omni_wheel_radius" value="0.04" />
   <xacro:property name="omni_wheel_height" value="0.04" />
-  <xacro:property name="omni_wheel_mass" value="0.7" /> <!-- in kg-->
+  <xacro:property name="omni_wheel_mass" value="0.15" /> <!-- in kg-->
   <xacro:macro name="cylinder_inertia" params="m r h">
     <inertia  ixx="${m*(3*r*r+h*h)/12}" ixy = "0" ixz = "0"
@@ -26,13 +26,13 @@
           <xacro:if value="${reflect}">
             <geometry>
-              <mesh filename="package://dextrobot_description/src/meshes/wheels/mechanum_wheel_1.dae" />
+              <mesh filename="package://dextrobot_description/src/mesh/wheels/mechanum_wheel_1.dae" scale="0.1 0.1 0.1"/>
             </geometry>
           </xacro:if>
           <xacro:unless value="${reflect}">
             <geometry>
-              <mesh filename="package://summit_xl_description/meshes/wheels/mechanum_wheel_2.dae" />
+              <mesh filename="package://dextrobot_description/src/mesh/wheels/mechanum_wheel_2.dae" scale="0.1 0.1 0.1"/>
             </geometry>
-		  </xacro:unless>
-        </xacro:if>
+		      </xacro:unless>
+          </xacro:if>
         <xacro:unless value="${hq}">
           <origin xyz="0 0 0" rpy="0 0 0" />
@@ -48,5 +48,5 @@
 				<origin xyz="0 0 0" rpy="${PI/2} 0 0" />
         <geometry>
-				<cylinder length="${omni_wheel_height}" radius="${omni_wheel_radius}" />
+				  <cylinder length="${omni_wheel_height}" radius="${omni_wheel_radius}" />
         </geometry>
       </collision>
