Commit message: tf parameters tuning

File: ROS/dextrobot_ws/src/dextrobot_description/src/robot/dextrobot.urdf.xacro (robot description, xacro)
@@ -15,18 +15,18 @@
 	<!-- Front Left -->
 	<xacro:property name="wheel_1_offset_x" value="-1" />    <!-- x,y,z in translation from base_link to the center of the wheel -->
-	<xacro:property name="wheel_1_offset_y" value="-0.8" />
-	<xacro:property name="wheel_1_offset_z" value="0.0" />
+	<xacro:property name="wheel_1_offset_y" value="0.65" />
+	<xacro:property name="wheel_1_offset_z" value="0" />
 	<!-- Front Right -->
 	<xacro:property name="wheel_2_offset_x" value="0.72" />    <!-- x,y,z in translation from base_link to the center of the wheel -->
-	<xacro:property name="wheel_2_offset_y" value="0.05" />
-	<xacro:property name="wheel_2_offset_z" value="0.0" />
+	<xacro:property name="wheel_2_offset_y" value="0.65" />
+	<xacro:property name="wheel_2_offset_z" value="0" />
 	<!-- Back Left -->
 	<xacro:property name="wheel_3_offset_x" value="-1" />    <!-- x,y,z in translation from base_link to the center of the wheel -->
-	<xacro:property name="wheel_3_offset_y" value="-2.2" />
-	<xacro:property name="wheel_3_offset_z" value="0.0" />
+	<xacro:property name="wheel_3_offset_y" value="-0.73" />
+	<xacro:property name="wheel_3_offset_z" value="0" />
 	<!-- Back Right -->
 	<xacro:property name="wheel_4_offset_x" value="0.72" />    <!-- x,y,z in translation from base_link to the center of the wheel -->
-	<xacro:property name="wheel_4_offset_y" value="-1.35" />
-	<xacro:property name="wheel_4_offset_z" value="0.0" />
+	<xacro:property name="wheel_4_offset_y" value="-0.73" />
+	<xacro:property name="wheel_4_offset_z" value="0" />
 	<!-- IMU parameters -->
 	<xacro:property name="imu_offset_x" value="0.229" />    <!-- x,y,z in translation from base_link to the center of the wheel -->
@@ -35,6 +35,6 @@
 	<!-- Camera parameters -->
 	<xacro:property name="camera_offset_x" value="-0.15" />    <!-- x,y,z in translation from base_link to the center of the wheel -->
-	<xacro:property name="camera_offset_y" value="-0.25" />
-	<xacro:property name="camera_offset_z" value="1.1" />
+	<xacro:property name="camera_offset_y" value="0.8" />
+	<xacro:property name="camera_offset_z" value="0.7" />
 	<!-- Sonar parameters -->
 	<!-- front sonar -->

File: ROS/dextrobot_ws/src/dextrobot_description/src/urdf/bases/dextrobot_base.urdf.xacro (robot description, xacro)
@@ -5,5 +5,5 @@
   <!-- Robot mechanical and motor parameters -->
   <xacro:property name="PI" value="3.1415926535897931"/>
-  <xacro:property name="wheel_radius" value="0.04" />
+  <xacro:property name="wheel_radius" value="0.4" />
 	<!-- BASE FOOTPRINT -->
 	  <xacro:if value="${publish_bf}">
@@ -25,5 +25,5 @@
   <link name="${prefix}base_link">
     <visual>
-      <origin xyz="2 0 0.1" rpy="${PI/2} 0 ${-PI/2}" />
+      <origin xyz="2 1.05 -0.3" rpy="${PI/2} 0 ${-PI/2}" />
       <xacro:if value="${hq}">
       <geometry>
@@ -41,5 +41,5 @@
     </visual>
     <collision>
-       <origin xyz="2 0 0.1" rpy="${PI/2} 0 ${-PI/2}" />
+       <origin xyz="2 1.05 -0.3" rpy="${PI/2} 0 ${-PI/2}" />
        <geometry>
          <mesh filename="package://dextrobot_description/src/mesh/base/dextrobot_chassis.dae" scale="0.01 0.01 0.01"/>

File: ROS/dextrobot_ws/src/dextrobot_description/src/urdf/wheels/omni_wheel.urdf.xacro (robot description, xacro)
@@ -16,5 +16,5 @@
       <child link="${prefix}_wheel_link"/>
       <xacro:insert_block name="origin" />
-      <axis xyz="0 1 0" rpy="0 0 0" />
+      <axis xyz="1 0 0"/>
       <limit effort="100" velocity="100"/>
       <joint_properties damping="0.0" friction="0.0"/>
@@ -23,5 +23,5 @@
       <visual>
         <xacro:if value="${hq}">
-          <origin xyz="0 0 0" rpy="0 0 0" />
+          <origin xyz="0 -0.425 -0.42" rpy="0 0 0" />
           <xacro:if value="${reflect}">
             <geometry>

Commit message: uniform the unit of measurement

File: ROS/dextrobot_ws/src/dextrobot_description/src/robot/dextrobot.urdf.xacro (robot description, xacro)
@@ -14,43 +14,43 @@
 	<!-- Wheel parameters -->
 	<!-- Front Left -->
-	<xacro:property name="wheel_1_offset_x" value="-1" />    <!-- x,y,z in translation from base_link to the center of the wheel -->
-	<xacro:property name="wheel_1_offset_y" value="0.65" />
+	<xacro:property name="wheel_1_offset_x" value="-0.1" />    <!-- x,y,z in translation from base_link to the center of the wheel -->
+	<xacro:property name="wheel_1_offset_y" value="0.065" />
 	<xacro:property name="wheel_1_offset_z" value="0" />
 	<!-- Front Right -->
-	<xacro:property name="wheel_2_offset_x" value="0.72" />    <!-- x,y,z in translation from base_link to the center of the wheel -->
-	<xacro:property name="wheel_2_offset_y" value="0.65" />
+	<xacro:property name="wheel_2_offset_x" value="0.072" />    <!-- x,y,z in translation from base_link to the center of the wheel -->
+	<xacro:property name="wheel_2_offset_y" value="0.065" />
 	<xacro:property name="wheel_2_offset_z" value="0" />
 	<!-- Back Left -->
-	<xacro:property name="wheel_3_offset_x" value="-1" />    <!-- x,y,z in translation from base_link to the center of the wheel -->
-	<xacro:property name="wheel_3_offset_y" value="-0.73" />
+	<xacro:property name="wheel_3_offset_x" value="-0.1" />    <!-- x,y,z in translation from base_link to the center of the wheel -->
+	<xacro:property name="wheel_3_offset_y" value="-0.073" />
 	<xacro:property name="wheel_3_offset_z" value="0" />
 	<!-- Back Right -->
-	<xacro:property name="wheel_4_offset_x" value="0.72" />    <!-- x,y,z in translation from base_link to the center of the wheel -->
-	<xacro:property name="wheel_4_offset_y" value="-0.73" />
+	<xacro:property name="wheel_4_offset_x" value="0.072" />    <!-- x,y,z in translation from base_link to the center of the wheel -->
+	<xacro:property name="wheel_4_offset_y" value="-0.073" />
 	<xacro:property name="wheel_4_offset_z" value="0" />
 	<!-- IMU parameters -->
-	<xacro:property name="imu_offset_x" value="0.229" />    <!-- x,y,z in translation from base_link to the center of the wheel -->
-	<xacro:property name="imu_offset_y" value="0.235" />
+	<xacro:property name="imu_offset_x" value="0.0229" />    <!-- x,y,z in translation from base_link to the center of the wheel -->
+	<xacro:property name="imu_offset_y" value="0.0235" />
 	<xacro:property name="imu_offset_z" value="0.0" />
 	<!-- Camera parameters -->
-	<xacro:property name="camera_offset_x" value="-0.15" />    <!-- x,y,z in translation from base_link to the center of the wheel -->
-	<xacro:property name="camera_offset_y" value="0.8" />
-	<xacro:property name="camera_offset_z" value="0.7" />
+	<xacro:property name="camera_offset_x" value="-0.015" />    <!-- x,y,z in translation from base_link to the center of the wheel -->
+	<xacro:property name="camera_offset_y" value="0.08" />
+	<xacro:property name="camera_offset_z" value="0.07" />
 	<!-- Sonar parameters -->
 	<!-- front sonar -->
-	<xacro:property name="front_sonar_offset_x" value="0.229" />    <!-- x,y,z in translation from base_link to the center of the wheel -->
-	<xacro:property name="front_sonar_offset_y" value="0.235" />
+	<xacro:property name="front_sonar_offset_x" value="0.0229" />    <!-- x,y,z in translation from base_link to the center of the wheel -->
+	<xacro:property name="front_sonar_offset_y" value="0.0235" />
 	<xacro:property name="front_sonar_offset_z" value="0.0" />
 	<!-- left sonar -->
-	<xacro:property name="left_sonar_offset_x" value="0.229" />    <!-- x,y,z in translation from base_link to the center of the wheel -->
-	<xacro:property name="left_sonar_offset_y" value="0.235" />
+	<xacro:property name="left_sonar_offset_x" value="0.0229" />    <!-- x,y,z in translation from base_link to the center of the wheel -->
+	<xacro:property name="left_sonar_offset_y" value="0.0235" />
 	<xacro:property name="left_sonar_offset_z" value="0.0" />
 	<!-- right sonar -->
-	<xacro:property name="right_sonar_offset_x" value="0.229" />    <!-- x,y,z in translation from base_link to the center of the wheel -->
-	<xacro:property name="right_sonar_offset_y" value="0.235" />
+	<xacro:property name="right_sonar_offset_x" value="0.0229" />    <!-- x,y,z in translation from base_link to the center of the wheel -->
+	<xacro:property name="right_sonar_offset_y" value="0.0235" />
 	<xacro:property name="right_sonar_offset_z" value="0.0" />
 	<!-- back sonar -->
-	<xacro:property name="back_sonar_offset_x" value="0.229" />    <!-- x,y,z in translation from base_link to the center of the wheel -->
-	<xacro:property name="back_sonar_offset_y" value="0.235" />
+	<xacro:property name="back_sonar_offset_x" value="0.0229" />    <!-- x,y,z in translation from base_link to the center of the wheel -->
+	<xacro:property name="back_sonar_offset_y" value="0.0235" />
 	<xacro:property name="back_sonar_offset_z" value="0.0" />
 	<!-- Flag to select the high or low quality model -->
@@ -68,5 +68,5 @@
   			<origin xyz="${wheel_1_offset_x} ${wheel_1_offset_y} ${wheel_1_offset_z}" rpy="0 0 0"/>
   		</xacro:omni_wheel>
-  		<xacro:omni_wheel prefix="$(arg prefix)front_right" parent="$(arg prefix)base_link" reflect="false" hq="${hq}">
+  		<xacro:omni_wheel prefix="$(arg prefix)front_right" parent="$(arg prefix)base_link" reflect="true" hq="${hq}">
   			<origin xyz="${wheel_2_offset_x} ${wheel_2_offset_y} ${wheel_2_offset_z}" rpy="0 0 ${PI}"/>
   		</xacro:omni_wheel>

File: ROS/dextrobot_ws/src/dextrobot_description/src/urdf/bases/dextrobot_base.urdf.xacro (robot description, xacro)
@@ -5,5 +5,5 @@
   <!-- Robot mechanical and motor parameters -->
   <xacro:property name="PI" value="3.1415926535897931"/>
-  <xacro:property name="wheel_radius" value="0.4" />
+  <xacro:property name="wheel_radius" value="0.04" />
 	<!-- BASE FOOTPRINT -->
 	  <xacro:if value="${publish_bf}">
@@ -25,13 +25,13 @@
   <link name="${prefix}base_link">
     <visual>
-      <origin xyz="2 1.05 -0.3" rpy="${PI/2} 0 ${-PI/2}" />
+      <origin xyz="0.2 0.105 -0.03" rpy="${PI/2} 0 ${-PI/2}" />
       <xacro:if value="${hq}">
       <geometry>
-      <mesh filename="package://dextrobot_description/src/mesh/base/dextrobot_chassis.STL" scale="0.01 0.01 0.01"/>
+      <mesh filename="package://dextrobot_description/src/mesh/base/dextrobot_chassis.STL" scale="0.001 0.001 0.001"/>
       </geometry>
       </xacro:if>
       <xacro:unless value="${hq}">
       <geometry>
-      <mesh filename="package://dextrobot_description/src/mesh/base/dextrobot_chassis.dae" scale="0.01 0.01 0.01"/>
+      <mesh filename="package://dextrobot_description/src/mesh/base/dextrobot_chassis.dae" scale="0.001 0.001 0.001"/>
       </geometry>
       </xacro:unless>
@@ -41,7 +41,7 @@
     </visual>
     <collision>
-       <origin xyz="2 1.05 -0.3" rpy="${PI/2} 0 ${-PI/2}" />
+       <origin xyz="0.2 0.105 -0.03" rpy="${PI/2} 0 ${-PI/2}" />
        <geometry>
-         <mesh filename="package://dextrobot_description/src/mesh/base/dextrobot_chassis.dae" scale="0.01 0.01 0.01"/>
+         <mesh filename="package://dextrobot_description/src/mesh/base/dextrobot_chassis.dae" scale="0.001 0.001 0.001"/>
        </geometry>
     </collision>

File: ROS/dextrobot_ws/src/dextrobot_description/src/urdf/wheels/omni_wheel.urdf.xacro (robot description, xacro)
@@ -3,6 +3,6 @@
   <xacro:property name="M_PI" value="3.1415926535897931" />
   <!-- Wheels -->
-  <xacro:property name="omni_wheel_radius" value="0.04" />
-  <xacro:property name="omni_wheel_height" value="0.04" />
+  <xacro:property name="omni_wheel_radius" value="0.04" /> <!-- in m-->
+  <xacro:property name="omni_wheel_height" value="0.04" /> <!-- in m-->
   <xacro:property name="omni_wheel_mass" value="0.15" /> <!-- in kg-->
   <xacro:macro name="cylinder_inertia" params="m r h">
@@ -23,13 +23,13 @@
       <visual>
         <xacro:if value="${hq}">
-          <origin xyz="0 -0.425 -0.42" rpy="0 0 0" />
+          <origin xyz="0 -0.0425 -0.042" rpy="0 0 0" />
           <xacro:if value="${reflect}">
             <geometry>
-              <mesh filename="package://dextrobot_description/src/mesh/wheels/mechanum_wheel_1.dae" scale="0.1 0.1 0.1"/>
+              <mesh filename="package://dextrobot_description/src/mesh/wheels/mechanum_wheel_1.dae" scale="0.01 0.01 0.01"/>
             </geometry>
           </xacro:if>
           <xacro:unless value="${reflect}">
             <geometry>
-              <mesh filename="package://dextrobot_description/src/mesh/wheels/mechanum_wheel_2.dae" scale="0.1 0.1 0.1"/>
+              <mesh filename="package://dextrobot_description/src/mesh/wheels/mechanum_wheel_2.dae" scale="0.01 0.01 0.01"/>
             </geometry>
 		      </xacro:unless>

Commit message: added frames for sonar and imu sensor

File: ROS/dextrobot_ws/src/dextrobot_description/src/robot/dextrobot.urdf.xacro (robot description, xacro)
@@ -30,28 +30,11 @@
 	<xacro:property name="wheel_4_offset_z" value="0" />
 	<!-- IMU parameters -->
-	<xacro:property name="imu_offset_x" value="0.0229" />    <!-- x,y,z in translation from base_link to the center of the wheel -->
-	<xacro:property name="imu_offset_y" value="0.0235" />
-	<xacro:property name="imu_offset_z" value="0.0" />
+	<xacro:property name="imu_offset_x" value="0" />    <!-- x,y,z in translation from base_link to the center of the wheel -->
+	<xacro:property name="imu_offset_y" value="0" />
+	<xacro:property name="imu_offset_z" value="0.05" />
 	<!-- Camera parameters -->
 	<xacro:property name="camera_offset_x" value="-0.015" />    <!-- x,y,z in translation from base_link to the center of the wheel -->
 	<xacro:property name="camera_offset_y" value="0.08" />
 	<xacro:property name="camera_offset_z" value="0.07" />
-	<!-- Sonar parameters -->
-	<!-- front sonar -->
-	<xacro:property name="front_sonar_offset_x" value="0.0229" />    <!-- x,y,z in translation from base_link to the center of the wheel -->
-	<xacro:property name="front_sonar_offset_y" value="0.0235" />
-	<xacro:property name="front_sonar_offset_z" value="0.0" />
-	<!-- left sonar -->
-	<xacro:property name="left_sonar_offset_x" value="0.0229" />    <!-- x,y,z in translation from base_link to the center of the wheel -->
-	<xacro:property name="left_sonar_offset_y" value="0.0235" />
-	<xacro:property name="left_sonar_offset_z" value="0.0" />
-	<!-- right sonar -->
-	<xacro:property name="right_sonar_offset_x" value="0.0229" />    <!-- x,y,z in translation from base_link to the center of the wheel -->
-	<xacro:property name="right_sonar_offset_y" value="0.0235" />
-	<xacro:property name="right_sonar_offset_z" value="0.0" />
-	<!-- back sonar -->
-	<xacro:property name="back_sonar_offset_x" value="0.0229" />    <!-- x,y,z in translation from base_link to the center of the wheel -->
-	<xacro:property name="back_sonar_offset_y" value="0.0235" />
-	<xacro:property name="back_sonar_offset_z" value="0.0" />
 	<!-- Flag to select the high or low quality model -->
 	<xacro:property name="hq" value="true" />
@@ -63,5 +46,5 @@
 		<!-- *************** -->
 		<!-- Here we create the robot elements using the xacro:macros imported at the beggining of this file -->
-		<!-- Summit XL base -->
+		<!-- Dextrobot base -->
 		<xacro:dextrobot_base prefix="$(arg prefix)" publish_bf="true" hq="${hq}" />
 		<xacro:omni_wheel prefix="$(arg prefix)front_left" parent="$(arg prefix)base_link" reflect="false" hq="${hq}">
@@ -79,5 +62,5 @@
         <!-- IMU -->
 		<xacro:sensor_imu_hector prefix="$(arg prefix)imu" parent="$(arg prefix)base_link">
-			<origin xyz="${imu_offset_x} ${imu_offset_y} ${imu_offset_z}" rpy="0 0 0"/>
+			<origin xyz="${imu_offset_x} ${imu_offset_y} ${imu_offset_z}" rpy="0 0 ${PI/2}"/>
 		</xacro:sensor_imu_hector>
 	    <!-- RGBD -->

File: ROS/dextrobot_ws/src/dextrobot_description/src/urdf/bases/dextrobot_base.urdf.xacro (robot description, xacro)
@@ -6,4 +6,21 @@
   <xacro:property name="PI" value="3.1415926535897931"/>
   <xacro:property name="wheel_radius" value="0.04" />
+  <!-- Sonar parameters -->
+	<!-- front sonar -->
+	<xacro:property name="front_sonar_offset_x" value="0.0" />    <!-- x,y,z in translation from base_link to the center of the wheel -->
+	<xacro:property name="front_sonar_offset_y" value="0.1" />
+	<xacro:property name="front_sonar_offset_z" value="0.0" />
+	<!-- left sonar -->
+	<xacro:property name="left_sonar_offset_x" value="-0.09" />    <!-- x,y,z in translation from base_link to the center of the wheel -->
+	<xacro:property name="left_sonar_offset_y" value="0.0" />
+	<xacro:property name="left_sonar_offset_z" value="0.0" />
+	<!-- right sonar -->
+	<xacro:property name="right_sonar_offset_x" value="0.06" />    <!-- x,y,z in translation from base_link to the center of the wheel -->
+	<xacro:property name="right_sonar_offset_y" value="0.0" />
+	<xacro:property name="right_sonar_offset_z" value="0.0" />
+	<!-- back sonar -->
+	<xacro:property name="back_sonar_offset_x" value="0.0" />    <!-- x,y,z in translation from base_link to the center of the wheel -->
+	<xacro:property name="back_sonar_offset_y" value="-0.1" />
+	<xacro:property name="back_sonar_offset_z" value="0.0" />
 	<!-- BASE FOOTPRINT -->
 	  <xacro:if value="${publish_bf}">
@@ -47,4 +64,60 @@
     </collision>
   </link>
+  <!-- FRONT SONAR SENSOR -->
+  <link name="${prefix}front_sonar">
+		  <visual>
+			  <origin xyz="0 0 0" rpy="0 0 0" />
+			  <geometry>
+				 <box size="0.001 0.001 0.001" />
+			  </geometry>
+		  </visual>
+	</link>
+  <joint name="${prefix}front_sonar_joint" type="fixed">
+		<origin xyz="${front_sonar_offset_x} ${front_sonar_offset_y} ${front_sonar_offset_z}" rpy="0 0 ${PI/2}" />
+		<parent link="${prefix}base_link"/>
+		<child link="${prefix}front_sonar"/>
+	</joint>
+  <!-- LEFT SONAR SENSOR -->
+  <link name="${prefix}left_sonar">
+		  <visual>
+			  <origin xyz="0 0 0" rpy="0 0 0" />
+			  <geometry>
+				 <box size="0.001 0.001 0.001" />
+			  </geometry>
+		  </visual>
+	</link>
+  <joint name="${prefix}left_sonar_joint" type="fixed">
+		<origin xyz="${left_sonar_offset_x} ${left_sonar_offset_y} ${left_sonar_offset_z}" rpy="0 0 ${PI}" />
+		<parent link="${prefix}base_link"/>
+		<child link="${prefix}left_sonar"/>
+	</joint>
+  <!-- RIGHT SONAR SENSOR -->
+  <link name="${prefix}right_sonar">
+		  <visual>
+			  <origin xyz="0 0 0" rpy="0 0 0" />
+			  <geometry>
+				 <box size="0.001 0.001 0.001" />
+			  </geometry>
+		  </visual>
+	</link>
+  <joint name="${prefix}right_sonar_joint" type="fixed">
+		<origin xyz="${right_sonar_offset_x} ${right_sonar_offset_y} ${right_sonar_offset_z}" rpy="0 0 0" />
+		<parent link="${prefix}base_link"/>
+		<child link="${prefix}right_sonar"/>
+	</joint>
+  <!-- BACK SONAR SENSOR -->
+  <link name="${prefix}back_sonar">
+		  <visual>
+			  <origin xyz="0 0 0" rpy="0 0 0" />
+			  <geometry>
+				 <box size="0.001 0.001 0.001" />
+			  </geometry>
+		  </visual>
+	</link>
+  <joint name="${prefix}back_sonar_joint" type="fixed">
+		<origin xyz="${back_sonar_offset_x} ${back_sonar_offset_y} ${back_sonar_offset_z}" rpy="0 0 -${PI/2}" />
+		<parent link="${prefix}base_link"/>
+		<child link="${prefix}back_sonar"/>
+	</joint>
   </xacro:macro>
 </robot>
